File: RPLIDARA1_USB_Adapter/RPLIDARA1_USB_Adapter.kicad_pcb (KiCad board)
At the start: 2 copper layers, 38 x 21.5 mm, 24 parts, among them J1 USB_B_Micro, J2 Molex SPOX 5268-07A, J3 Pin headers 1.54mm 01x08, U2 CP2102N-A02-GQFN28

Commit message: Modified texts
Routing:
- net GND: vias 41 -> 40
Changed lines of the file:
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@@
     (effects (font (size 0.7 0.7) (thickness 0.1)) (justify left mirror))
   )
-  (gr_text "5V" (at 82.35 91.875 90) (layer "B.Mask")
+  (gr_text "5V" (at 82.6 91.875 90) (layer "B.Mask")
     (effects (font (size 0.7 0.7) (thickness 0.1)) (justify mirror))
   )
@@
     (effects (font (size 0.7 0.7) (thickness 0.1)) (justify left mirror))
   )
-  (gr_text "3V3" (at 82.35 81.715 90) (layer "B.Mask")
+  (gr_text "3V3" (at 82.6 81.715 90) (layer "B.Mask")
     (effects (font (size 0.7 0.7) (thickness 0.1)) (justify mirror))
   )
@@
     (effects (font (size 0.7 0.7) (thickness 0.1)) (justify left mirror))
   )
-  (gr_text "CTS" (at 82.35 89.335 90) (layer "B.Mask")
+  (gr_text "CTS" (at 82.6 89.335 90) (layer "B.Mask")
     (effects (font (size 0.7 0.7) (thickness 0.1)) (justify mirror))
   )
-  (gr_text "GND" (at 82.35 74.095 90) (layer "B.Mask")
+  (gr_text "GND" (at 82.6 74.095 90) (layer "B.Mask")
     (effects (font (size 0.7 0.7) (thickness 0.1)) (justify mirror))
   )
-  (gr_text "DTR" (at 82.35 86.795 90) (layer "B.Mask")
+  (gr_text "DTR" (at 82.6 86.795 90) (layer "B.Mask")
     (effects (font (size 0.7 0.7) (thickness 0.1)) (justify mirror))
   )
@@
     (effects (font (size 0.7 0.7) (thickness 0.1)) (justify left mirror))
   )
-  (gr_text "TXD" (at 82.35 76.635 90) (layer "B.Mask")
+  (gr_text "TXD" (at 82.6 76.635 90) (layer "B.Mask")
     (effects (font (size 0.7 0.7) (thickness 0.1)) (justify mirror))
   )
-  (gr_text "RXD" (at 82.35 79.175 90) (layer "B.Mask")
+  (gr_text "RXD" (at 82.6 79.175 90) (layer "B.Mask")
     (effects (font (size 0.7 0.7) (thickness 0.1)) (justify mirror))
   )
-  (gr_text "RTS" (at 82.35 84.255 90) (layer "B.Mask")
+  (gr_text "RTS" (at 82.6 84.255 90) (layer "B.Mask")
     (effects (font (size 0.7 0.7) (thickness 0.1)) (justify mirror))
   )
@@
   (via (at 101 85.5) (size 0.7) (drill 0.4) (layers "F.Cu" "B.Cu") (net 2))
   (via (at 113 92.5) (size 0.7) (drill 0.4) (layers "F.Cu" "B.Cu") (net 2))
-  (via (at 96.35 73.95) (size 0.7) (drill 0.4) (layers "F.Cu" "B.Cu") (net 2))
   (via (at 104.075 81.825) (size 0.7) (drill 0.4) (layers "F.Cu" "B.Cu") (net 2))
   (via (at 114.3 87.825) (size 0.7) (drill 0.4) (layers "F.Cu" "B.Cu") (net 2))
@@
   (arc (start 102.107322 82.282322) (mid 102.120405 82.301902) (end 102.125 82.325) (width 0.5) (layer "F.Cu") (net 3))
   (arc (start 101.275 83.3) (mid 101.191925 83.355508) (end 101.093933 83.375) (width 0.3) (layer "F.Cu") (net 3))
-  (segment (start 97.375 73.744255) (end 97.375 78.575) (width 0.5) (layer "B.Cu") (net 3))
+  (segment (start 97.375 78.575) (end 97.375 74.77904) (width 0.5) (layer "B.Cu") (net 3))
+  (segment (start 85.775 74.96996) (end 85.775 79.353961) (width 0.5) (layer "B.Cu") (net 3))
   (segment (start 101.832107 81.332107) (end 101.692893 81.192893) (width 0.5) (layer "B.Cu") (net 3))
-  (segment (start 85.775 79.353961) (end 85.775 74.96996) (width 0.5) (layer "B.Cu") (net 3))
-  (segment (start 87.96248 72.975) (end 96.69332 72.975) (width 0.5) (layer "B.Cu") (net 3))
-  (segment (start 84.1 81.715) (end 85.289897 80.525103) (width 0.5) (layer "B.Cu") (net 3))
+  (segment (start 85.289897 80.525103) (end 84.1 81.715) (width 0.5) (layer "B.Cu") (net 3))
   (segment (start 97.375 79.518439) (end 97.375 78.575) (width 0.5) (layer "B.Cu") (net 3))
   (segment (start 102.125 82.35) (end 102.125 82.039214) (width 0.5) (layer "B.Cu") (net 3))
   (segment (start 100.985786 80.9) (end 98.747601 80.9) (width 0.5) (layer "B.Cu") (net 3))
+  (segment (start 95.508778 72.975) (end 87.96248 72.975) (width 0.5) (layer "B.Cu") (net 3))
   (segment (start 97.812752 80.512752) (end 97.76855 80.46855) (width 0.5) (layer "B.Cu") (net 3))
-  (arc (start 85.289897 80.525103) (mid 85.648926 79.987778) (end 85.775 79.353961) (width 0.5) (layer "B.Cu") (net 3))
-  (arc (start 86.319444 73.655556) (mid 85.916496 74.25861) (end 85.775 74.96996) (width 0.5) (layer "B.Cu") (net 3))
+  (arc (start 85.775 79.353961) (mid 85.648926 79.987778) (end 85.289897 80.525103) (width 0.5) (layer "B.Cu") (net 3))
   (arc (start 101.692893 81.192893) (mid 101.36847 80.97612) (end 100.985786 80.9) (width 0.5) (layer "B.Cu") (net 3))
-  (arc (start 97.131501 73.156501) (mid 96.930462 73.022171) (end 96.69332 72.975) (width 0.5) (layer "B.Cu") (net 3))
   (arc (start 97.812752 80.512752) (mid 98.241685 80.799367) (end 98.747601 80.9) (width 0.5) (layer "B.Cu") (net 3))
   (arc (start 97.76855 80.46855) (mid 97.47728 80.032636) (end 97.375 79.518439) (width 0.5) (layer "B.Cu") (net 3))
+  (arc (start 86.319444 73.655556) (mid 85.916496 74.25861) (end 85.775 74.96996) (width 0.5) (layer "B.Cu") (net 3))
+  (arc (start 96.859478 73.534478) (mid 96.239772 73.120404) (end 95.508778 72.975) (width 0.5) (layer "B.Cu") (net 3))
   (arc (start 87.96248 72.975) (mid 87.073264 73.151876) (end 86.319444 73.655556) (width 0.5) (layer "B.Cu") (net 3))
-  (arc (start 97.131501 73.156501) (mid 97.311736 73.426205) (end 97.375 73.744255) (width 0.5) (layer "B.Cu") (net 3))
+  (arc (start 96.859478 73.534478) (mid 97.241024 74.105496) (end 97.375 74.77904) (width 0.5) (layer "B.Cu") (net 3))
   (arc (start 102.125 82.039214) (mid 102.04888 81.656531) (end 101.832107 81.332107) (width 0.5) (layer "B.Cu") (net 3))
   (segment (start 98.525 80.6) (end 98.525 80.683577) (width 0.3) (layer "F.Cu") (net 4))
