File: Lipo_BMS/Lipo_BMS.kicad_pcb (KiCad board)
At the start: 2 copper layers, 90 x 37 mm, 80 parts, among them J1 Deans connector male, J102 B4B-XH-A(LF)(SN), J103 B4B-XH-A(LF)(SN), J2 XT30, J3 STL1550/2G-3.5, J4 54-00286, J5 Terminal block, J6 B3B-PH-SM4-TB(LF)(SN), J7 XT30, Q101 SI4459ADY-T1-GE3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

Commit message: Added BOM to LiPo board
Parts:
- added kibuzzard-643EEDF5: G***, kibuzzard-643EEDF5, F.Cu at (131.7, 77.4)
- added kibuzzard-643EEE0C: G***, kibuzzard-643EEE0C, F.Cu at (132.9, 81.1)
- U2: value MAX17263xxTE -> MAX17263LETD+T
Routing:
- net /SCL: track 66.2 -> 66.9 mm
- net GND: vias 70 -> 74

Commit message: added via in pad for fuse for anti-shear
Routing:
- net Net-(BAR101C-A): track 32.5 -> 34.1 mm, vias 3 -> 2
